File: pcb/WaterBlaster/PowerProtection.kicad_sch (KiCad schematic)
At the start: 13 parts, among them J2 Conn_01x03, U3 R-78E5.0-0.5, U7 AZ1117EH-3.3TRG1

Commit message: Updating firmware and CAD
Parts:
- renumbered C9 to C1, C10 to C2, C8 to C3, C7 to C4, F2 to F1, J2 to J15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
