File: pcb/WaterBlaster/WaterBlasterV2/WaterBlasterV2/PowerProtection.kicad_sch (KiCad schematic)
At the start: 16 parts, among them J1 Conn_01x03, U1 R-78E5.0-0.5

Commit message: V2 Firmware
Other:
- note added: "Add fuse on 5V here- for the V2 boards, bodged in series with the inductor on the oversized footprint - required to fuse transducer"
Changed lines of the file:
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@@
 	(generator_version "9.0")
 	(paper "A4")
+	(text "Add fuse on 5V here- for the V2 boards, bodged in series with the inductor on the oversized footprint - required to fuse transducer"
+		(exclude_from_sim no)
+		(at 80.772 36.83 0)
+		(effects
+			(font
+				(size 1.27 1.27)
+			)
+		)
+	)
 	(junction
 		(at 207.01 53.34)
